File: pcb/imu/imu.sch (EAGLE design)
At the start: 0 parts

Commit message: Add components to MPU breakout. Needs board layout and revision
Parts:
- added C1, C4: 0.1u, SparkFun-Passives:CAP0805
- added C2, C6: 10n, SparkFun-Passives:CAP0805
- added C3: 2.2n, SparkFun-Passives:CAP0805
- added C5, C7: 4.7u, SparkFun-Passives:CAP0805
- added JP1: (no value), SparkFun-Connectors:M05SMD2
- added LED1: (no value), SparkFun-LED:LED0603
- added R1, R2, R3, R4: 10k, SparkFun-Passives:RESISTOR0805-RES
- added R5: 150, SparkFun-Passives:RESISTOR0805-RES
- added SJ1, SJ2: JUMPER-PAD-2-NC_BY_TRACE, SparkFun-Passives:JUMPER-PAD-2-NC_BY_TRACE
- added SJ3: JUMPER-PAD-3-2OF3_NC_BY_TRACE_SMALL, SparkFun-Passives:JUMPER-PAD-3-2OF3_NC_BY_TRACE_SMALL
- added U1: (no value), SparkFun-Sensors:MPU-9150QFN-24-NP
- added U2: V_REG_LDOSMD2, SparkFun-PowerIC:V_REG_LDOSMD2
Connections:
- new net AD0: SJ3.2, U1.AD0
- new net CLKOUT: U1.CLKOUT
- new net ESCL: R3.1, U1.E_SCL
- new net ESDA: R4.1, U1.E_SDA
- new net GND: C1.2, C2.2, C3.2, C4.2, C5.2, C6.2, C7.2, JP1.3, LED1.C, SJ1.1, SJ2.1, SJ3.3, U1.GND@15, U1.GND@17, U1.GND@18, U2.GND
- new net INT: U1.INT
- new net N$1: LED1.A, R5.2
- new net N$3: SJ1.2, U1.FSYNC
- new net N$4: C3.1, U1.CPOUT
- new net N$5: C4.1, U1.REGOUT
- new net N$6: SJ2.2, U1.CLKIN
- new net N$7: C6.1, U2.BP
- new net SCL: JP1.4, R2.1, U1.SCL
- new net SDA: JP1.5, R1.1, U1.SDA
- new net VCC: C1.1, C2.1, C7.1, JP1.2, R1.2, R2.2, R3.2, R4.2, R5.1, SJ3.1, U1.VDD@13, U1.VDD@3, U1.VLOGIC, U2.OUT
- new net VIN: C5.1, JP1.1, U2.EN, U2.IN
