File: pcb/imu/imu.sch (EAGLE design)
At the start: 19 parts, among them U2 V_REG_LDOSMD2

Commit message: Change LED to 0805 package
Parts:
- LED1: device SparkFun-LED:LED0603 -> SparkFun-LED:LED0805
Changed lines of the file:
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@@
 <setting verticaltext="up"/>
 </settings>
-<grid distance="0.1" unitdist="inch" unit="inch" style="lines" multiple="1" display="yes" altdistance="0.01" altunitdist="inch" altunit="inch"/>
+<grid distance="0.1" unitdist="inch" unit="inch" style="lines" multiple="1" display="no" altdistance="0.01" altunitdist="inch" altunit="inch"/>
 <layers>
 <layer number="1" name="Top" color="4" fill="1" visible="no" active="no"/>
@@
 <part name="SJ3" library="SparkFun-Passives" deviceset="JUMPER-PAD-3-2OF3_NC_BY_TRACE" device="_SMALL"/>
 <part name="GND7" library="SparkFun-Aesthetics" deviceset="GND" device=""/>
-<part name="LED1" library="SparkFun-LED" deviceset="LED" device="0603"/>
+<part name="LED1" library="SparkFun-LED" deviceset="LED" device="0805"/>
 <part name="U2" library="SparkFun-PowerIC" deviceset="V_REG_LDO" device="SMD2"/>
 <part name="GND8" library="SparkFun-Aesthetics" deviceset="GND" device=""/>

Commit message: Finish MPU board layout revision 1
Parts:
- removed R3, R4: 10k, SparkFun-Passives:RESISTOR0805-RES
- removed U2: V_REG_LDOSMD2, SparkFun-PowerIC:V_REG_LDOSMD2
- added 3V3_REG: V_REG_LDOSMD, SparkFun-PowerIC:V_REG_LDOSMD
- C6*: value 10n -> 470p
- renumbered C5 to C5*, C6 to C6*, LED1 to PWR, SJ1 to FSYNC, SJ2 to CLKIN, SJ3 to ADDRESS, U1 to MPU9150
Connections:
- net ESCL: no longer R3.1
- net ESDA: no longer R4.1
- net GND: now also 3V3_REG.GND; no longer U2.GND
- net N$7: now also 3V3_REG.BP; no longer U2.BP
- net VCC: now also 3V3_REG.OUT; no longer R3.2, R4.2, U2.OUT
- net VIN: now also 3V3_REG.EN, 3V3_REG.IN; no longer U2.EN, U2.IN

Commit message: MPU revision 2 with 3mm holes
Parts:
- removed CLKIN, FSYNC: JUMPER-PAD-2-NC_BY_TRACE, SparkFun-Passives:JUMPER-PAD-2-NC_BY_TRACE
Connections:
- removed net N$3: FSYNC.2, MPU9150.FSYNC
- removed net N$6: CLKIN.2, MPU9150.CLKIN
- net GND: now also MPU9150.CLKIN, MPU9150.FSYNC; no longer CLKIN.1, FSYNC.1
- net SCL: now also JP1.5; no longer JP1.4
- net SDA: now also JP1.4; no longer JP1.5
Changed lines of the file:
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@@
 <part name="GND3" library="SparkFun-Aesthetics" deviceset="GND" device=""/>
 <part name="GND4" library="SparkFun-Aesthetics" deviceset="GND" device=""/>
-<part name="FSYNC" library="SparkFun-Passives" deviceset="JUMPER-PAD-2-NC_BY_TRACE" device="" value="JUMPER-PAD-2-NC_BY_TRACE"/>
-<part name="CLKIN" library="SparkFun-Passives" deviceset="JUMPER-PAD-2-NC_BY_TRACE" device="" value="JUMPER-PAD-2-NC_BY_TRACE"/>
-<part name="GND5" library="SparkFun-Aesthetics" deviceset="GND" device=""/>
 <part name="GND6" library="SparkFun-Aesthetics" deviceset="GND" device=""/>
 <part name="ADDRESS" library="SparkFun-Passives" deviceset="JUMPER-PAD-3-2OF3_NC_BY_TRACE" device="_SMALL"/>
@@
 <instance part="GND3" gate="1" x="93.98" y="109.22"/>
 <instance part="GND4" gate="1" x="106.68" y="109.22"/>
-<instance part="FSYNC" gate="G$1" x="66.04" y="116.84" smashed="yes" rot="R90">
-<attribute name="NAME" x="63.5" y="114.3" size="1.778" layer="95" rot="R90"/>
-</instance>
-<instance part="CLKIN" gate="G$1" x="78.74" y="116.84" smashed="yes" rot="R90">
-<attribute name="NAME" x="76.2" y="114.3" size="1.778" layer="95" rot="R90"/>
-</instance>
-<instance part="GND5" gate="1" x="66.04" y="106.68"/>
-<instance part="GND6" gate="1" x="78.74" y="106.68"/>
+<instance part="GND6" gate="1" x="78.74" y="119.38"/>
 <instance part="ADDRESS" gate="G$1" x="218.44" y="142.24" smashed="yes">
 <attribute name="NAME" x="220.98" y="142.621" size="1.778" layer="95"/>
@@
 </segment>
 <segment>
-<pinref part="FSYNC" gate="G$1" pin="1"/>
-<wire x1="66.04" y1="111.76" x2="66.04" y2="109.22" width="0.1524" layer="91"/>
-<pinref part="GND5" gate="1" pin="GND"/>
-</segment>
-<segment>
-<pinref part="CLKIN" gate="G$1" pin="1"/>
-<wire x1="78.74" y1="111.76" x2="78.74" y2="109.22" width="0.1524" layer="91"/>
-<pinref part="GND6" gate="1" pin="GND"/>
-</segment>
-<segment>
 <pinref part="ADDRESS" gate="G$1" pin="3"/>
 <pinref part="GND7" gate="1" pin="GND"/>
@@
 <pinref part="C6*" gate="G$1" pin="2"/>
 <pinref part="GND12" gate="1" pin="GND"/>
+</segment>
+<segment>
+<pinref part="MPU9150" gate="G$1" pin="CLKIN"/>
+<wire x1="129.54" y1="124.46" x2="78.74" y2="124.46" width="0.1524" layer="91"/>
+<wire x1="78.74" y1="124.46" x2="78.74" y2="121.92" width="0.1524" layer="91"/>
+<pinref part="GND6" gate="1" pin="GND"/>
+<pinref part="MPU9150" gate="G$1" pin="FSYNC"/>
+<wire x1="129.54" y1="127" x2="78.74" y2="127" width="0.1524" layer="91"/>
+<wire x1="78.74" y1="127" x2="78.74" y2="124.46" width="0.1524" layer="91"/>
 </segment>
 </net>
@@
 </segment>
 <segment>
-<pinref part="JP1" gate="G$1" pin="5"/>
-<wire x1="182.88" y1="78.74" x2="167.64" y2="78.74" width="0.1524" layer="91"/>
-<label x="167.64" y="78.74" size="1.778" layer="95" rot="MR0" xref="yes"/>
+<pinref part="JP1" gate="G$1" pin="4"/>
+<wire x1="182.88" y1="81.28" x2="177.8" y2="81.28" width="0.1524" layer="91"/>
+<label x="177.8" y="81.28" size="1.778" layer="95" rot="MR0" xref="yes"/>
 </segment>
 </net>
@@
 </segment>
 <segment>
-<pinref part="JP1" gate="G$1" pin="4"/>
-<wire x1="182.88" y1="81.28" x2="175.26" y2="81.28" width="0.1524" layer="91"/>
-<label x="175.26" y="81.28" size="1.778" layer="95" rot="MR0" xref="yes"/>
+<pinref part="JP1" gate="G$1" pin="5"/>
+<wire x1="182.88" y1="78.74" x2="170.18" y2="78.74" width="0.1524" layer="91"/>
+<label x="170.18" y="78.74" size="1.778" layer="95" rot="MR0" xref="yes"/>
 </segment>
 </net>
@@
 </segment>
 </net>
-<net name="N$3" class="0">
-<segment>
-<pinref part="MPU9150" gate="G$1" pin="FSYNC"/>
-<pinref part="FSYNC" gate="G$1" pin="2"/>
-<wire x1="129.54" y1="127" x2="66.04" y2="127" width="0.1524" layer="91"/>
-<wire x1="66.04" y1="127" x2="66.04" y2="121.92" width="0.1524" layer="91"/>
-</segment>
-</net>
-<net name="N$6" class="0">
-<segment>
-<pinref part="MPU9150" gate="G$1" pin="CLKIN"/>
-<pinref part="CLKIN" gate="G$1" pin="2"/>
-<wire x1="129.54" y1="124.46" x2="78.74" y2="124.46" width="0.1524" layer="91"/>
-<wire x1="78.74" y1="124.46" x2="78.74" y2="121.92" width="0.1524" layer="91"/>
-</segment>
-</net>

Commit message: Finalise IMU board schematic/layout. Try to make 3D model (*.emn/emp) files
Parts:
- 3V3_REG: value V_REG_LDOSMD -> (none); device SparkFun-PowerIC:V_REG_LDOSMD -> SparkFun-PowerIC:MIC52053.3V
Other:
- moved on the sheet: 3V3_REG, ADDRESS, C1, C2, C3, C4, C5*, C6*, C7, JP1, MPU9150, PWR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
